Commit message: Bugfixing

File: test_3dof.urdf (robot description, URDF)
Before this commit: robot lbr_iiwa, 5 links, 4 joints
Joints:
- joint joint3: origin xyz=1 0 0 rpy=0 0 0 -> xyz=1 0 0 rpy=1.57079632679489661923 0 0
- joint joint4: origin xyz=1 0 0 rpy=-1.57079632679489661923 0 0 -> xyz=1 0 0 rpy=0 0 0

Commit message: Added more stuff

File: test_3dof.urdf (robot description, URDF)
Before this commit: robot lbr_iiwa, 5 links, 4 joints
Joints:
- joint joint1: origin xyz=0 0 8 rpy=0 0 0 -> xyz=0 0 0 rpy=0 0 0

Commit message: Added functionality to influence plotting

File: test_3dof.urdf (robot description, URDF)
Before this commit: robot myrobot, 5 links, 4 joints
Links:
- link world: geometry visual box size=0.25 0.25 1
Joints:
- joint joint1: origin xyz=0 0 0 rpy=0 0 0 -> xyz=0 0 0.5 rpy=0 0 0

Commit message: Bugfixing

File: test_3dof.urdf (robot description, URDF)
Before this commit: robot myrobot, 5 links, 4 joints
Links:
- link world: geometry 
