Commit message: Almost there

File: model/hexapod.urdf (robot description, URDF)
Before this commit: robot hexapod, 27 links, 26 joints
Links:
- added link world
Joints:
- added joint wold_base_link: type prismatic, parent world, child base_link, origin xyz=0 0 0 rpy=0 0 0, axis 0 0 1, limit lower=-300000 upper=3000000 effort=150 velocity=150000000

Commit message: Collision checking with arbitrary robots

File: model/hexapod.urdf (robot description, URDF)
Before this commit: robot hexapod, 28 links, 27 joints
Joints:
- removed joint wold_base_link
- added joint a0: type prismatic, parent world, child base_link, origin xyz=0 0 0 rpy=0 0 0, axis 0 0 1, limit lower=-300000 upper=3000000 effort=150 velocity=150000000
