Commit message: Dunno

File: model/block_model.urdf (robot description, URDF)
Before this commit: robot myrobot, 3 links, 2 joints
Links:
- removed link link1
- removed link link2
- added link base_link, mass 1; collision box size=1 1 1; visual box size=1 1 1
- added link front_left_coxa, mass 1; collision box size=1 0.15 0.15; visual box size=1 0.15 0.15
- added link front_left_femour, mass 1; collision box size=1 0.15 0.15; visual box size=1 0.15 0.15
- added link front_left_tibia, mass 1; collision box size=1 0.15 0.15; visual box size=1 0.15 0.15
- added link front_right_coxa, mass 1; collision box size=1 0.15 0.15; visual box size=1 0.15 0.15
Joints:
- removed joint joint1
- removed joint joint2
- added joint joint00: type fixed, parent world, child base_link, origin xyz=0 0 0 rpy=0 0 0, axis 0 0 0, limit lower=-300000 upper=3000000 effort=150 velocity=150000000
- added joint joint01: type revolute, parent base_link, child front_left_coxa, origin xyz=0.5 0 0 rpy=0 0 0, axis 0 0 1, limit lower=-300000 upper=3000000 effort=150 velocity=150000000
- added joint joint02: type revolute, parent front_left_coxa, child front_left_femour, origin xyz=1 0 0 rpy=0 0 0, axis 0 1 0, limit lower=-300000 upper=3000000 effort=150 velocity=150000000
- added joint joint03: type revolute, parent front_left_femour, child front_left_tibia, origin xyz=1 0 0 rpy=0 0 0, axis 0 1 0, limit lower=-300000 upper=3000000 effort=150 velocity=150000000
- added joint joint04: type revolute, parent base_link, child front_right_coxa, origin xyz=0 0.5 0 rpy=0 0 1.57079632679489661923, axis 0 0 1, limit lower=-300000 upper=3000000 effort=150 velocity=150000000

File: model/hexapod.urdf (robot description, URDF)
Before this commit: robot hexapod, 28 links, 27 joints
Joints:
- removed joint a0
- removed joint base_link_square
- removed joint front_left_body_coxa
- removed joint front_left_coxa_femour
- removed joint front_left_femour_tibia
- removed joint front_left_tibia_virtual
- removed joint front_right_body_coxa
- removed joint front_right_coxa_femour
- removed joint front_right_femour_tibia
- removed joint front_right_tibia_virtual
- removed joint middle_left_body_coxa
- removed joint middle_left_coxa_femour
- removed joint middle_left_femour_tibia
- removed joint middle_left_tibia_virtual
- removed joint middle_right_body_coxa
- removed joint middle_right_coxa_femour
- removed joint middle_right_femour_tibia
- removed joint middle_right_tibia_virtual
- removed joint rear_left_body_coxa
- removed joint rear_left_coxa_femour
- removed joint rear_left_femour_tibia
- removed joint rear_left_tibia_virtual
- removed joint rear_right_body_coxa
- removed joint rear_right_coxa_femour
- removed joint rear_right_femour_tibia
- removed joint rear_right_tibia_virtual
- removed joint square_sensor_link
- added joint j01: type revolute, parent base_link, child front_left_coxa, origin xyz=0.1205 0.0705 0 rpy=0.0 0.0 0.785398163397, axis 0 0 1, limit lower=-300000 upper=3000000 effort=150 velocity=150000000
- added joint j02: type revolute, parent base_link, child front_right_coxa, origin xyz=0.1205 -0.0705 0 rpy=0.0 0.0 -0.785398163397, axis 0 0 1, limit lower=-2.4 upper=2.4 effort=10 velocity=3.14159265359
- added joint j03: type revolute, parent base_link, child middle_left_coxa, origin xyz=0.0 0.1131 0 rpy=0.0 0.0 1.57079632679, axis 0 0 1, limit lower=-2.4 upper=2.4 effort=10 velocity=3.14159265359
- added joint j04: type revolute, parent base_link, child middle_right_coxa, origin xyz=0.0 -0.1131 0.0 rpy=0.0 0.0 -1.57079632679, axis 0 0 1, limit lower=-2.4 upper=2.4 effort=10 velocity=3.14159265359
- added joint j05: type revolute, parent base_link, child rear_left_coxa, origin xyz=-0.1205 0.0705 0 rpy=0.0 0.0 2.35619449019, axis 0 0 1, limit lower=-2.4 upper=2.4 effort=10 velocity=3.14159265359
- added joint j06: type revolute, parent base_link, child rear_right_coxa, origin xyz=-0.1205 -0.0705 0 rpy=0.0 0.0 -2.35619449019, axis 0 0 1, limit lower=-2.4 upper=2.4 effort=10 velocity=3.14159265359
- added joint j07: type revolute, parent front_left_coxa, child front_left_femour, origin xyz=0.06 0 0 rpy=1.57079632679489661923 0.0 0.0, axis 0 0 1, limit lower=-300000 upper=3000000 effort=150 velocity=150000000
- added joint j08: type revolute, parent front_right_coxa, child front_right_femour, origin xyz=0.06 0 0 rpy=-1.57079632679489661923 0.0 0.0, axis 0 0 1, limit lower=-2.4 upper=2.4 effort=10 velocity=3.14159265359
- added joint j09: type revolute, parent middle_left_coxa, child middle_left_femour, origin xyz=0.06 0 0 rpy=1.57079632679489661923 0.0 0.0, axis 0 0 1, limit lower=-2.4 upper=2.4 effort=10 velocity=3.14159265359
- added joint j10: type revolute, parent middle_right_coxa, child middle_right_femour, origin xyz=0.06 0 0 rpy=-1.57079632679489661923 0.0 0.0, axis 0 0 1, limit lower=-2.4 upper=2.4 effort=10 velocity=3.14159265359
- added joint j11: type revolute, parent rear_left_coxa, child rear_left_femour, origin xyz=0.06 0 0 rpy=1.57079632679489661923 0.0 0.0, axis 0 0 1, limit lower=-2.4 upper=2.4 effort=10 velocity=3.14159265359
- added joint j12: type revolute, parent rear_right_coxa, child rear_right_femour, origin xyz=0.06 0 0 rpy=-1.57079632679489661923 0.0 0.0, axis 0 0 1, limit lower=-2.4 upper=2.4 effort=10 velocity=3.14159265359
- added joint j13: type revolute, parent front_left_femour, child front_left_tibia, origin xyz=0.0836 0 0 rpy=0.0 0.0 0.0, axis 0 0 1, limit lower=-2.4 upper=2.4 effort=10 velocity=3.14159265359
- added joint j14: type revolute, parent front_right_femour, child front_right_tibia, origin xyz=0.0836 0 0 rpy=0.0 0.0 0.0, axis 0 0 1, limit lower=-2.4 upper=2.4 effort=10 velocity=3.14159265359
- added joint j15: type revolute, parent middle_left_femour, child middle_left_tibia, origin xyz=0.0836 0 0 rpy=0.0 0.0 0.0, axis 0 0 1, limit lower=-2.4 upper=2.4 effort=10 velocity=3.14159265359
- added joint j16: type revolute, parent middle_right_femour, child middle_right_tibia, origin xyz=0.0836 0 0 rpy=0.0 0.0 0.0, axis 0 0 1, limit lower=-2.4 upper=2.4 effort=10 velocity=3.14159265359
- added joint j17: type revolute, parent rear_left_femour, child rear_left_tibia, origin xyz=0.0836 0 0 rpy=0.0 0.0 0.0, axis 0 0 1, limit lower=-2.4 upper=2.4 effort=10 velocity=3.14159265359
- added joint j18: type revolute, parent rear_right_femour, child rear_right_tibia, origin xyz=0.0836 0 0 rpy=0.0 0.0 0.0, axis 0 0 1, limit lower=-2.4 upper=2.4 effort=10 velocity=3.14159265359
- added joint j19: type fixed, parent front_left_tibia, child front_left_end_effector, origin xyz=0.2 0 0 rpy=0.0 0.0 0.0, axis 0 0 1, limit lower=-2.4 upper=2.4 effort=10 velocity=3.14159265359
- added joint j20: type fixed, parent front_right_tibia, child front_right_end_effector, origin xyz=0.2 0 0 rpy=0.0 0.0 0.0, axis 0 0 1, limit lower=-2.4 upper=2.4 effort=10 velocity=3.14159265359
- added joint j21: type fixed, parent middle_left_tibia, child middle_left_end_effector, origin xyz=0.2 0 0 rpy=0.0 0.0 0.0, axis 0 0 1, limit lower=-2.4 upper=2.4 effort=10 velocity=3.14159265359
- added joint j22: type fixed, parent middle_right_tibia, child middle_right_end_effector, origin xyz=0.2 0 0 rpy=0.0 0.0 0.0, axis 0 0 1, limit lower=-2.4 upper=2.4 effort=10 velocity=3.14159265359
- added joint j23: type fixed, parent rear_left_tibia, child rear_left_end_effector, origin xyz=0.2 0 0 rpy=0.0 0.0 0.0, axis 0 0 1, limit lower=-2.4 upper=2.4 effort=10 velocity=3.14159265359
- added joint j24: type fixed, parent rear_right_tibia, child rear_right_end_effector, origin xyz=0.2 0 0 rpy=0.0 0.0 0.0, axis 0 0 1, limit lower=-2.4 upper=2.4 effort=10 velocity=3.14159265359
- added joint j25: type fixed, parent world, child base_link, origin xyz=0 0 0.16 rpy=0 0 0, axis 0 0 1, limit lower=-300000 upper=3000000 effort=150 velocity=150000000
- added joint k00: type fixed, parent base_link, child square, origin xyz=0.1205 0 0 rpy=0.0 0.0 0.0
- added joint k01: type fixed, parent square, child sensor_link, origin xyz=0.025 0 0 rpy=0.0 0.0 0.0

Commit message: Implemented contact constraints

File: model/block_model.urdf (robot description, URDF)
Before this commit: robot myrobot, 6 links, 5 joints
Links:
- added link front_left_end_effector, mass 0; collision box size=0.0001 0.15 0.15; visual box size=0.0001 0.15 0.15
Joints:
- added joint joint05: type revolute, parent base_link, child front_right_coxa, origin xyz=0 0.5 0 rpy=0 0 1.57079632679489661923, axis 0 0 1, limit lower=-300000 upper=3000000 effort=150 velocity=150000000
- joint joint00: origin xyz=0 0 0 rpy=0 0 0 -> xyz=0 0 2 rpy=0 0 0
- joint joint04: axis 0 0 1 -> 0 1 0; child front_right_coxa -> front_left_end_effector; origin xyz=0 0.5 0 rpy=0 0 1.57079632679489661923 -> xyz=1 0 0 rpy=0 0 0; parent base_link -> front_left_tibia; type revolute -> fixed
